Commit message: Update simple_car.urdf

File: urdf/simple_car.urdf (robot description, URDF)
Before this commit: robot simple_car, 5 links, 4 joints
Links:
- link base_link: geometry visual box size=0.6 0.3 0.15
- link front_left_wheel: geometry visual cylinder length=0.02 radius=0.05
- link front_right_wheel: geometry visual cylinder length=0.02 radius=0.05
- link rear_left_wheel: geometry visual cylinder length=0.02 radius=0.05
- link rear_right_wheel: geometry visual cylinder length=0.02 radius=0.05
Joints:
- removed joint front_left_joint
- removed joint front_right_joint
- removed joint rear_left_joint
- removed joint rear_right_joint
- added joint joint_front_left: type fixed, parent base_link, child front_left_wheel, origin xyz=0.2 0.15 -0.05
- added joint joint_front_right: type fixed, parent base_link, child front_right_wheel, origin xyz=0.2 -0.15 -0.05
- added joint joint_rear_left: type fixed, parent base_link, child rear_left_wheel, origin xyz=-0.2 0.15 -0.05
- added joint joint_rear_right: type fixed, parent base_link, child rear_right_wheel, origin xyz=-0.2 -0.15 -0.05
